File: MAAV_Projects/Spine/14v0/Spine14_v0.sch (EAGLE design)
At the start: 31 parts, among them Q1 BSS138, Q2 MOSFET-NCHANNELBSS138, Q3 MOSFET-NCHANNELBSS138, Q4 MOSFET-NCHANNELBSS138, U1 ATMEGA328-AU

Commit message: power management systems for Spine14v0
Parts:
- added C1, C10, C12, C5, C7: 0.1uF, rcl:C-USC0603
- added C11: 4.7uF, rcl:C-USC0805
- added C13, C9: 1.0uF, rcl:C-USC0603
- added C14: 2.2uF, rcl:C-USC0603
- added C15, C16: 24pF, rcl:C-USC0603
- added C17, C18: 10pF, rcl:C-USC0603
- added C2, C6, C8: 0.01uF, rcl:C-USC0603
- added C4: 10nF, rcl:C-USC0603
- added IC1: PINTO_SMD, MAAV:PINTO_SMD
- added Q5: (no value), crystal:CRYSTALTC26H
- added Q6: (no value), crystal:CRYSTALHC49UP
- added R11: 470, rcl:R-US_R0603
- added R13: 250k, rcl:R-US_R0603
- added R9: 10k, rcl:R-US_R0603
- added S1: P498_SWITCH-OFF-MOM, MAAV_13v1:P498_SWITCH-OFF-MOM
- added U2: REG_3V_8SOIC, MAAV:REG_3V_8SOIC
- U$2: value GUMSTIX_PINTO -> JON_LIB_MAX3221-RS232; device GUMSTIX_PINTO:GUMSTIX_PINTO -> MAAV_13v1:JON_LIB_MAX3221-RS232
Connections:
- removed net N$8: U$2.GPIO67
- removed net N$9: U$2.GPIO168
- new net +3V3: C11.1, C2.1, C5.1, C6.1, C7.1, C8.1, C9.1, R13.2, R9.2, U$3.VBAT, U$3.VDD@1, U$3.VDD@2, U$3.VDD@3, U$3.VDD@4, U$3.VDDA, U2.OUT, U2.OUT2
- new net N$12: R11.1, S1.P1, S1.P3
- new net T_GNDX: U$3.GNDX
- new net T_OSC0: C18.1, Q6.2, U$3.OSC0
- new net T_OSC1: C17.1, Q6.1, U$3.OSC1
- new net T_RESET: C4.1, R11.2, R9.1
- new net T_VDDC: C1.1, C12.1, C13.1, C14.1
- new net T_XOSC0: C15.2, Q5.2, U$3.XOSC0
- new net T_XOSC1: C16.1, Q5.1, U$3.XOSC1
- net +5V: now also C10.1, U2.IN, U2.IN2
- net GND: now also C1.2, C10.2, C11.2, C12.2, C13.2, C14.2, C17.2, C18.2, C2.2, C4.2, C5.2, C6.2, C7.2, C8.2, C9.2, S1.P2, S1.P4, U$3.GND@1, U$3.GND@2, U$3.GND@3, U$3.GND@4, U$3.GNDA, U2./EN, U2.GND
- net N$10: now also R13.1, U2.PG; no longer U$2.GPIO64
- net N$7: now also C15.1, C16.2; no longer U$2.GPIO66
- net SCL_1V8: now also IC1.GPIO184/SCL; no longer U$2.SCL3
- net SDA_1V8: now also IC1.GPIO185/SDA; no longer U$2.SDA3
Other:
- note added: "3V3 Power Supply"
- note added: "5V Power Supply"
- note added: "Communications with External Computer/Sensor Hardware"
- note added: "Power Management"
- note added: "Power Supplies"
- note removed: "Power Supply"

Commit message: added JTAG programmer for tiva and nets for ATMega
Parts:
- removed IC1: PINTO_SMD, MAAV:PINTO_SMD
- added C25, C26, C27, C28: 100nF, Jon_LIB:C-EUC0603
- added C29, C30: 22pF, Jon_LIB:C-EUC0603
- added IC2: PINTO_SMD, MAAV:PINTO_SMD
- added ICDI_JTAG: TC2050-IDC-NL, MAAV:TC2050-IDC-NL
- added LED1: GREEN, MAAV_13v1:JON_LIB_LEDCHIPLED_0603
- added Q8: CRYSTAL_16MHZ_SMD, Jon_LIB:CRYSTAL_16MHZ_SMD
- added R12, R15: 10k, rcl:R-US_R0603
- added R14: 10k, Jon_LIB:R-USR0603
- added R16: 330, rcl:R-US_R0603
- added S3: SWITCH-OFF-MOM, p498:SWITCH-OFF-MOM
- added SV1: (no value), Jon_LIB:AVRISP-63X2_SMD
- added SV5, SV6: (no value), Jon_LIB:MA03-1
- Q5: value (none) -> 32.768KHz
- Q6: value (none) -> 16MHz
- U1: DIGIKEY# (none) -> ATMEGA328-AU-ND
Connections:
- new net BATT_SENSE: U1.ADC6
- new net ICDI_TCK: ICDI_JTAG.TCK, R12.1, U$3.PC0/TCK/SWCLK
- new net ICDI_TDI: ICDI_JTAG.TDI, U$3.PC2/TDI
- new net ICDI_TDO: ICDI_JTAG.TDO, U$3.PC3/TDO/SWO
- new net ICDI_TMS: ICDI_JTAG.TMS, R15.1, U$3.PC1/TMS/SWDIO
- new net KILL_SIG: SV5.3, U1.(ADC0)PC0
- new net LED1: U1.(OC1)PB1
- new net LED2: U1.(ICP)PB0
- new net LED3: U1.(T0)PD4
- new net MISO: SV1.MISO, U1.(MISO)PB4
- new net MOSI: SV1.MOSI, U1.(MOSI)PB3
- new net MOTOR_LOGIC: U1.(AIN1)PD7
- new net N$13: C27.1, U1.AREF
- new net N$14: C29.2, Q8.P$2, U1.XTAL2
- new net N$15: C30.2, Q8.P$1, U1.XTAL1
- new net N$39: U1.(AIN0)PD6
- new net N$8: LED1.A, R16.1
- new net RESET: R14.1, S3.P1, S3.P3, SV1.RESET, U1.RESET
- new net SCK: SV1.SCK, U1.(SCK)PB5
- new net SCL_5V: U1.(ADC5)PC5
- new net SDA_5V: U1.(ADC4)PC4
- new net SERVO_1: SV6.3
- net +3V3: now also R12.2, R15.2, R16.2
- net +5V: now also C25.1, C26.1, C28.1, R14.2, SV1.VCC, SV5.2, SV6.2, U1.AVCC, U1.VCC, U1.VCC2
- net GND: now also C25.2, C26.2, C27.2, C28.2, C29.1, C30.1, ICDI_JTAG.GND, LED1.C, S3.P2, S3.P4, SV1.GND, SV5.1, SV6.1, U1.AGND, U1.GND, U1.GND2
- net SCL_1V8: now also IC2.GPIO184/SCL; no longer IC1.GPIO184/SCL
- net SDA_1V8: now also IC2.GPIO185/SDA; no longer IC1.GPIO185/SDA
- net T_RESET: now also ICDI_JTAG.RST
Other:
- note added: "ATMega 328-AU"
- note added: "Gumtix Pinto"
- note added: "ICDI JTAG Programmer"
- note added: "Tiva TM4C123GH6PMI"

Commit message: most connections for gunstix, atmega, tiva, and power management systems. need to connect MCU's together and create motor output. consider phoenix edge lite
Parts:
- removed C26, C27: 100nF, Jon_LIB:C-EUC0603
- removed C29, C30: 22pF, Jon_LIB:C-EUC0603
- removed IC2: PINTO_SMD, MAAV:PINTO_SMD
- removed Q8: CRYSTAL_16MHZ_SMD, Jon_LIB:CRYSTAL_16MHZ_SMD
- removed S3: SWITCH-OFF-MOM, p498:SWITCH-OFF-MOM
- removed SV6: (no value), Jon_LIB:MA03-1
- removed U$2: JON_LIB_MAX3221-RS232, MAAV_13v1:JON_LIB_MAX3221-RS232
- added C19, C20: 22pF, Jon_LIB:C-EUC0603
- added C21, C22, C23, C24: 100nF, Jon_LIB:C-EUC0603
- added C37, C41: 0.1uF, Jon_LIB:C-EUC0603
- added C38, C39, C40: 0.47uF, Jon_LIB:C-EUC0805
- added IC3: PINTO_SMD, Jon_LIB:PINTO_SMD
- added J7: MA04-1, Jon_LIB:MA04-1
- added JP2: (no value), SparkFun-Connectors:M03PTH
- added LED2, LED3, LED4: GREEN, Jon_LIB:LEDCHIPLED_0603
- added MOUT1: MINI_FIT_JR_5569, SAUVE:MINI_FIT_JR_5569
- added N-FET1: MOSFET-NCHANNELBSS138, SparkFun-DiscreteSemi:MOSFET-NCHANNELBSS138
- added P-FET1: MOSFET_P-CHANNEL, SAUVE:MOSFET_P-CHANNEL
- added Q7: CRYSTAL_16MHZ_SMD, Jon_LIB:CRYSTAL_16MHZ_SMD
- added R17, R39: 10k, Jon_LIB:R-USR0603
- added R40: 432, Jon_LIB:R-USR0603
- added R44, R47, R48: 750, Jon_LIB:R-USR0805
- added S2: SWITCH-OFF-MOM, p498:SWITCH-OFF-MOM
- added U$11: MAX3221-RS232, Jon_LIB:MAX3221-RS232
- added U$4: JON_LIB_SWITCH_DPDT, MAAV_13v1:JON_LIB_SWITCH_DPDT
- added V_BATT: JON_LIB_BATTERY5A, MAAV_13v1:JON_LIB_BATTERY5A
- C25: value 100nF -> 10uF; device Jon_LIB:C-EUC0603 -> Jon_LIB:C-EUC1206; DIGIKEY# 1276-1000-1-ND -> 587-2399-1-ND
- R14: device Jon_LIB:R-USR0603 -> SparkFun-Resistors:RESISTOR0603-RES; DIGIKEY (none) -> RMCF0603JT10K0CT-ND; DIGIKEY# P10.0KHCT-ND -> (none)
- SV1: device Jon_LIB:AVRISP-63X2_SMD -> MAAV:AVRISP-63X2_PLUG_OF_NAILS
Connections:
- removed net ENABLE: U$1.ENA
- removed net N$39: U1.(AIN0)PD6
- removed net SERVO_1: SV6.3
- removed net VIN: IN_BY.1, IN_BY2.1, IN_BY3.1, U$1.VIN
- new net +1V8: IC3.VCC_1V8(1), IC3.VCC_1V8(2)
- new net A_*VCC: C22.1, C23.1, C24.1, U1.AVCC, U1.VCC, U1.VCC2
- new net A_AREF: C21.1, U1.AREF
- new net A_GND: C22.2, C23.2, C24.2, U1.AGND, U1.GND, U1.GND2
- new net A_RESET: R17.1, S2.P1, S2.P3, U1.RESET
- new net A_XTAL1: C20.2, Q7.P$1, U1.XTAL1
- new net A_XTAL2: C19.2, Q7.P$2, U1.XTAL2
- new net G_BATT_SENSE: IC3.ADCIN4, R39.1, R40.2
- new net G_V_BATT: C25.1, C28.1, IC3.V_BATT
- new net MOTOR0_PWM_1V8: IC3.GPIO147/PWM8
- new net MOTOR1_PWM_1V8: IC3.GPIO144/PWM9
- new net MOTOR2_PWM_1V8: IC3.GPIO145/PWM10
- new net MOTOR3_PWM_1V8: IC3.GPIO146/PWM11
- new net N$11: C37.1, U$11.C1+
- new net N$16: N-FET1.D, P-FET1.G, R14.1
- new net N$17: MOUT1.1, N-FET1.S
- new net N$32: C37.2, U$11.C1-
- new net N$33: LED3.A, R47.1
- new net N$34: LED4.A, R48.1
- new net N$35: C38.1, U$11.C2+
- new net N$36: C38.2, U$11.C2-
- new net N$9: LED2.A, R44.1
- new net ON/OFF: U$1.ENA, U$4.P$2
- new net POWER: R39.2, U$4.P$5
- new net RS-232_RX1: J7.P$3, U$11.RIN
- new net RS-232_TX1: J7.P$2, U$11.DOUT
- new net RX1_1V8: IC3.GPIO151/RXD1
- new net RX1_5V: U$11.ROUT
- new net TX1_1V8: IC3.GPIO148/TXD1
- new net TX1_5V: U$11.DIN
- new net V_BATT: IN_BY.1, IN_BY2.1, IN_BY3.1, U$1.VIN, U$4.P$6, V_BATT.BATT
- net +5V: now also C39.2, C41.1, J7.P$1, R17.2, U$11.FORCEOFF, U$11.VCC; no longer C25.1, C26.1, C28.1, R14.2, SV6.2, U1.AVCC, U1.VCC, U1.VCC2
- net DATA: now also JP2.1
- net EN: now also N-FET1.G
- net GND: now also C19.1, C20.1, C21.2, C40.2, C41.2, IC3.AGND, IC3.GND(1), IC3.GND(2), IC3.GND(3), J7.P$4, JP2.3, LED2.C, LED3.C, LED4.C, R40.1, S2.P2, S2.P4, U$11.EN, U$11.FORCEON, U$11.GND, U$4.P$1, U$4.P$4, V_BATT.GND; no longer C26.2, C27.2, C29.1, C30.1, S3.P2, S3.P4, SV6.1, U1.AGND, U1.GND, U1.GND2
- net LED1: now also R48.2
- net LED2: now also R47.2
- net LED3: now also R44.2
- net N$13: now also C39.1, U$11.V+; no longer C27.1, U1.AREF
- net N$14: now also C40.1, U$11.V-; no longer C29.2, Q8.P$2, U1.XTAL2
- net N$15: now also MOUT1.2, P-FET1.D; no longer C30.2, Q8.P$1, U1.XTAL1
- net RESET: no longer R14.1, S3.P1, S3.P3, U1.RESET
- net SCL_1V8: now also IC3.GPIO184/SCL; no longer IC2.GPIO184/SCL
- net SDA_1V8: now also IC3.GPIO185/SDA; no longer IC2.GPIO185/SDA
- net VCC: now also P-FET1.S, R14.2
- net VDD: now also JP2.2
Other:
- note added: "AVRISP Programmer"
- note added: "Board Power Management Systems"
- note added: "Kill Switch Signal Receiver"
- note added: "LED Indicators"
- note added: "Motor Outputs"
- note added: "THE Power Switch"
- note added: "Use 0.5% or better precision resistors"
- note added: "V_BATT"
- note added: "V_BATT = 4S = 14.8V"
- note removed: "GUMSTIX"
- note removed: "Power Supplies"

Commit message: worked on schematic.. shifted sheets around for 13v1
Parts:
- removed ICDI_JTAG: TC2050-IDC-NL, MAAV:TC2050-IDC-NL
- added R18, R19, R20: 10k, rcl:R-US_R0603
- added R21: 432, rcl:R-US_R0603
- added U$2: JTAG-ARM_TC-10, MAAV:JTAG-ARM_TC-10
- S1: value P498_SWITCH-OFF-MOM -> SWITCH-OFF-MOM_SMD_TACTILE; device MAAV_13v1:P498_SWITCH-OFF-MOM -> MAAV:SWITCH-OFF-MOM_SMD_TACTILE
- S2: value SWITCH-OFF-MOM -> SWITCH-OFF-MOM_SMD_TACTILE; device p498:SWITCH-OFF-MOM -> MAAV:SWITCH-OFF-MOM_SMD_TACTILE; DIGIKEY# P11084SCT-ND -> (none)
- SV1: device MAAV:AVRISP-63X2_PLUG_OF_NAILS -> MAAV:AVRISP-6_3X2_PLUG_OF_NAILS
- V_BATT: value JON_LIB_BATTERY5A -> BATT-CONN-50A_MINI-FIT-SR_THRU-HOLE; device MAAV_13v1:JON_LIB_BATTERY5A -> MAAV:BATT-CONN-50A_MINI-FIT-SR_THRU-HOLE
Connections:
- net SCL_5V0 renamed SCL_3V3G
- net SDA_5V0 renamed SDA_3V3G
- removed net BATT_SENSE: U1.ADC6
- new net A_BATT_SENSE: R20.1, R21.2, U1.ADC6
- new net SCL_3V3: U$3.PD0
- new net SDA_3V3: U$3.PE5
- net +1V8: now also Q3.G, Q4.G, R5.1, R7.1
- net +3V3: now also R6.1, R8.1
- net +5V: no longer R6.1, R8.1
- net A_RESET: now also S2.P$1; no longer S2.P1, S2.P3
- net GND: now also R21.1, S1.P$2, S2.P$2, U$2.GND; no longer ICDI_JTAG.GND, S1.P2, S1.P4, S2.P2, S2.P4
- net ICDI_TCK: now also U$2.TCK; no longer ICDI_JTAG.TCK
- net ICDI_TDI: now also U$2.TDI; no longer ICDI_JTAG.TDI
- net ICDI_TDO: now also U$2.TDO; no longer ICDI_JTAG.TDO
- net ICDI_TMS: now also U$2.TMS; no longer ICDI_JTAG.TMS
- net LV: no longer Q3.G, Q4.G, R5.1, R7.1
- net N$12: now also S1.P$1; no longer S1.P1, S1.P3
- net POWER: now also R20.2
- net T_RESET: now also U$2.RESET; no longer ICDI_JTAG.RST
- net V_BATT: now also V_BATT.VCC; no longer V_BATT.BATT
Other:
- note added: "0.5% or better precision resistors"
- note removed: "V_BATT"
- moved on the sheet: C1, C12, C13, C14, C15, C16, C17, C18, C19, C2, C20, C21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

Commit message: organized components and implemented i2c bus. next is motors
Parts:
- removed JP1: (no value), SparkFun-Connectors:M03PTH
- removed MOUT: MINI_FIT_JR_5569, SAUVE:MINI_FIT_JR_5569
- removed N-FET, Q2: MOSFET-NCHANNELBSS138, SparkFun-DiscreteSemi:MOSFET-NCHANNELBSS138
- removed P-FET: MOSFET_P-CHANNEL, SAUVE:MOSFET_P-CHANNEL
- removed Q1: BSS138, SparkFun-DiscreteSemi:MOSFET-NCHANNELBSS138
- removed R10, R3, R4, R6, R8: 10K, SparkFun:RESISTOR0603-RES
- added I2C_1, I2C_2: CONN_HEADER_4POS_RIGHT_ANGLE_I2C, MAAV:CONN_HEADER_4POS_RIGHT_ANGLE_I2C
- added Q8, Q9: MOSFET-NCHANNELBSS138, SparkFun-DiscreteSemi:MOSFET-NCHANNELBSS138
- added R22, R23, R24, R25: 10K, SparkFun:RESISTOR0603-RES
- R1: device SparkFun-Resistors:RESISTOR0603-RES -> rcl:R-US_R0603; DIGIKEY RMCF0603JT10K0CT-ND -> (none)
- R19: value 10k -> 432
- R2: value 10K -> 432; device SparkFun:RESISTOR0603-RES -> rcl:R-US_R0603; DIGIKEY RMCF0603JT10K0CT-ND -> (none)
Connections:
- removed net A_BATT_SENSE: R20.1, R21.2, U1.ADC6
- removed net HV: R10.1, R4.1
- removed net HV-CH1: Q1.D, R4.2
- removed net HV-CH2: Q2.D, R10.2
- removed net LV: Q1.G, Q2.G, R2.1, R3.1
- removed net LV-CH1: Q1.S, R3.2
- removed net LV-CH2: Q2.S, R2.2
- removed net N$1: MOUT.2, P-FET.D
- removed net N$2: N-FET.D, P-FET.G, R1.1
- removed net N$3: MOUT.1, N-FET.S
- removed net SCL_3V3G: Q3.D, R6.2, U$3.PB2/I2C0SCL
- removed net SDA_3V3G: Q4.D, R8.2, U$3.PB3/I2C0SDA
- new net MOTOR_POWER: R1.1, R2.2, R20.1, R21.2, U1.ADC6
- new net T_BATT_SENSE: R18.1, R19.2
- net +3V3: now also Q8.G, Q9.G, R22.1, R24.1; no longer R6.1, R8.1
- net +5V: now also I2C_1.P$1, I2C_2.P$1, R23.1, R25.1
- net DATA: no longer JP1.1
- net EN: no longer N-FET.G
- net GND: now also I2C_1.P$4, I2C_2.P$4, R19.1, R2.1; no longer JP1.3
- net POWER: now also R1.2, R18.2
- net SCL_3V3: now also Q3.D, Q8.S, R22.2, U$3.PB2/I2C0SCL; no longer U$3.PD0
- net SCL_5V: now also I2C_1.P$2, I2C_2.P$2, Q8.D, R23.2
- net SDA_3V3: now also Q4.D, Q9.S, R24.2, U$3.PB3/I2C0SDA; no longer U$3.PE5
- net SDA_5V: now also I2C_1.P$3, I2C_2.P$3, Q9.D, R25.2
- net VCC: no longer P-FET.S, R1.2
- net VDD: no longer JP1.2
Other:
- note added: "I2C Bus"
- note added: "PX4 Connectors"
- note added: "SCL Line"
- note added: "SDA Line"
- note removed: "Universal Bi-Directional Level Shifter"
- note removed: "Use 0.5% or better precision resistors"

Commit message: blah
Parts:
- added MOUT2: MINI_FIT_JR_5569, SAUVE:MINI_FIT_JR_5569
- added P-FET2: MOSFET_P-CHANNEL, SAUVE:MOSFET_P-CHANNEL
- added Q1: MOSFET-NCHANNELBSS138, SparkFun-DiscreteSemi:MOSFET-NCHANNELBSS138
- added R3: 10k, rcl:R-US_R0603
- added R4: 10k, SparkFun-Resistors:RESISTOR0603-RES
- R2: value 432 -> 10k
Connections:
- removed net N$17: MOUT1.1, N-FET1.S
- new net N$1: Q1.D, R2.1
- new net N$2: N-FET1.D, R4.1
- net GND: now also MOUT1.1, MOUT2.1, N-FET1.S, Q1.S, R3.1; no longer R2.1
- net MOTOR_LOGIC: now also Q1.G, R3.2
- net MOTOR_POWER: now also P-FET2.G
- net N$16: now also R4.2; no longer N-FET1.D
- net POWER: now also P-FET2.S
Other:
- note removed: "60A Switched Motor Ouput"
- moved on the sheet: I2C_1, I2C_2, JP2, MOUT1, N-FET1, R14, R2

Commit message: too tired. will finish motors later
Connections:
- new net N$3: MOUT2.2
- net POWER: no longer P-FET2.S
- net V_BATT: now also P-FET2.S
Changed lines of the file:
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@@
 <segment>
 <wire x1="-30.48" y1="-20.24" x2="-30.477459375" y2="-37.46" width="0.1524" layer="91"/>
-<wire x1="-30.477459375" y1="-37.46" x2="-30.48" y2="-38.14" width="0.1524" layer="91"/>
+<wire x1="-30.477459375" y1="-37.46" x2="-30.48" y2="-38.1" width="0.1524" layer="91"/>
 <pinref part="P-FET1" gate="G$1" pin="D"/>
 <pinref part="MOUT1" gate="G$1" pin="2"/>
@@
 </segment>
 </net>
-<net name="POWER" class="0">
+<net name="N$3" class="0">
+<segment>
+<wire x1="22.86" y1="-25.4" x2="22.86" y2="-20.32" width="0.1524" layer="91"/>
+<pinref part="MOUT2" gate="G$1" pin="2"/>
+<wire x1="22.86" y1="-25.4" x2="27.94" y2="-25.4" width="0.1524" layer="91"/>
+</segment>
+</net>
+<net name="V_BATT" class="0">
 <segment>
 <label x="17.78" y="0" size="1.778" layer="95" rot="R180" xref="yes"/>
@@
 </segment>
 </net>
-<net name="N$3" class="0">
-<segment>
-<wire x1="27.94" y1="-25.4" x2="22.86" y2="-25.4" width="0.1524" layer="91"/>
-<wire x1="22.86" y1="-25.4" x2="22.86" y2="-20.32" width="0.1524" layer="91"/>
-</segment>
-</net>
